File: ceas_8051.kicad_pcb (KiCad board)
At the start: 2 copper layers, 47 parts, among them J1 Conn_01x02_Pin, J2 Conn_01x02_Pin, Q1 S8550, Q2 S8550, Q3 S8550, Q4 S8550, Q5 S8550, Q6 S8550, Q7 S8550, U1 AT89C2051-24P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

Commit message: Saved version
Shitty PCB
Parts:
- added REF**: MountingHole_2.2mm_M2_DIN965, MountingHole:MountingHole_2.2mm_M2_DIN965, F.Cu at (33.0, 25.7)
- added REF**: MountingHole_2.2mm_M2_DIN965, MountingHole:MountingHole_2.2mm_M2_DIN965, F.Cu at (119.9, 25.7)
- added REF**: MountingHole_2.2mm_M2_DIN965, MountingHole:MountingHole_2.2mm_M2_DIN965, F.Cu at (33.0, 83.3)
- added REF**: MountingHole_2.2mm_M2_DIN965, MountingHole:MountingHole_2.2mm_M2_DIN965, F.Cu at (119.9, 83.3)
- moved R2 62.8 mm to (57.9, 71.6), turned to 90 degrees
- moved R3 58.1 mm to (60.5, 71.6), turned to 90 degrees
- moved R15 53.8 mm to (107.7, 47.0), turned to -90 degrees
- moved R14 53.7 mm to (105.4, 47.0), turned to -90 degrees
- moved R4 53.5 mm to (63.0, 71.6), turned to 90 degrees
- moved R5 47.7 mm to (67.1, 71.6), turned to 90 degrees
- moved R12 45.8 mm to (110.0, 47.0), turned to -90 degrees
- moved R6 43.5 mm to (69.3, 71.6), turned to 90 degrees
- moved R13 42.1 mm to (103.1, 47.0), turned to -90 degrees
- moved R11 40.8 mm to (112.3, 47.0), turned to -90 degrees
- moved R10 40.0 mm to (114.6, 47.0), turned to -90 degrees
- moved R7 39.1 mm to (72.1, 71.6), turned to 90 degrees
- moved DS1 12.0 mm to (53.3, 39.9), turned to 90 degrees
- moved DS2 12.0 mm to (78.7, 39.9), turned to 90 degrees
- moved DS3 11.7 mm to (102.9, 39.6), turned to 90 degrees
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Routing:
- net +5V: track 0.00 -> 206.1 mm
- net Net-(DS1-Pad1): track 0.00 -> 149.5 mm
- net Net-(DS1-Pad3): track 0.00 -> 149.3 mm
- net Net-(DS1-Pad4): track 0.00 -> 113.8 mm
- net Net-(DS1-Pad7): track 0.00 -> 96.3 mm
- net Net-(DS1-Pad9): track 0.00 -> 94.1 mm
- net Net-(DS1-Pad6): track 0.00 -> 82.2 mm
- net Net-(DS1-Pad8): track 0.00 -> 77.9 mm
- net D2: track 0.00 -> 74.2 mm
- net D1: track 0.00 -> 67.7 mm
- net A8: track 0.00 -> 63.6 mm
- net D3: track 0.00 -> 59.4 mm
- net Net-(Q6-C): track 0.00 -> 47.6 mm
- net Net-(BZ1--): track 0.00 -> 37.8 mm
- net D4: track 0.00 -> 37.1 mm
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- added copper zone on B.Cu, net GND
- added copper zone on F.Cu, net GND
